File: RadioPowerProtection.sch (KiCad schematic (older format))
At the start: 15 parts, among them Q1 IRF4905, Q2 IRF4905, Q3 Q_PNP_BCE

Commit message: Fix PNP transistor
Signed-off-by: Andres Gongora <mail@andresgongora.com>
Parts:
- removed Q3: Q_PNP_BCE, Package_TO_SOT_SMD:SOT-23, symbol Device:Q_PNP_BCE
- added Q3: BC858CLT1G, Package_TO_SOT_SMD:SOT-23, symbol Device:Q_PNP_BEC
- Q1, Q2: value IRF4905 -> SQP50P03-07_GE3
- R1: value 0 -> 4k7
- R3: value 1k -> 470
Connections:
- net PowerBus: now also Q3.2 (E)
- net at D4.1 (K): now also Q3.1 (B)
- net at D2.2 (A), Q2.1 (G), R4.1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: now also Q3.3 (C)
Changed lines of the file:
@@
 P 2750 2600
 F 0 "R1" H 2820 2646 50  0000 L CNN
-F 1 "0" H 2820 2555 50  0000 L CNN
+F 1 "4k7" H 2820 2555 50  0000 L CNN
 F 2 "NicerFootprints:SMD_0805" V 2680 2600 50  0001 C CNN
 F 3 "~" H 2750 2600 50  0001 C CNN
@@
 P 6100 2100
 F 0 "Q2" V 6442 2100 50  0000 C CNN
-F 1 "IRF4905" V 6351 2100 50  0000 C CNN
+F 1 "SQP50P03-07_GE3 " V 6351 2100 50  0000 C CNN
 F 2 "NicerFootprints:TO-220-3_Horizontal_TabDown" H 6300 2025 50  0001 L CIN
 F 3 "http://www.infineon.com/dgdl/irf4905.pdf?fileId=5546d462533600a4015355e32165197c" H 6100 2100 50  0001 L CNN
@@
 P 2350 2100
 F 0 "Q1" V 2692 2100 50  0000 C CNN
-F 1 "IRF4905" V 2601 2100 50  0000 C CNN
+F 1 "SQP50P03-07_GE3 " V 2601 2100 50  0000 C CNN
 F 2 "NicerFootprints:TO-220-3_Horizontal_TabDown" H 2550 2025 50  0001 L CIN
 F 3 "http://www.infineon.com/dgdl/irf4905.pdf?fileId=5546d462533600a4015355e32165197c" H 2350 2100 50  0001 L CNN
@@
 Wire Wire Line
 	5650 2750 5650 2900
-Wire Wire Line
-	3100 2000 4950 2000
 Connection ~ 7500 2500
 Wire Wire Line
@@
 Wire Wire Line
 	7500 2000 9000 2000
-$Comp
-L Device:Q_PNP_BCE Q3
-U 1 1 5FBCA9AB
-P 4850 2200
-F 0 "Q3" H 5040 2154 50  0000 L CNN
-F 1 "Q_PNP_BCE" H 5040 2245 50  0000 L CNN
-F 2 "Package_TO_SOT_SMD:SOT-23" H 5050 2300 50  0001 C CNN
-F 3 "~" H 4850 2200 50  0001 C CNN
-	1    4850 2200
-	1    0    0    1
-$EndComp
-Connection ~ 4950 2000
-Wire Wire Line
-	4950 2000 5250 2000
 $Comp
 L NicerLibrary:D_Zener D4
@@
 P 4650 2750
 F 0 "R3" H 4720 2796 50  0000 L CNN
-F 1 "1k" H 4720 2705 50  0000 L CNN
+F 1 "470" H 4720 2705 50  0000 L CNN
 F 2 "NicerFootprints:SMD_0805" V 4580 2750 50  0001 C CNN
 F 3 "~" H 4650 2750 50  0001 C CNN
@@
 Wire Wire Line
 	2750 2400 3100 2400
+Wire Wire Line
+	3100 2000 4950 2000
+$Comp
+L Device:Q_PNP_BEC Q3
+U 1 1 5FC03C98
+P 4850 2200
+F 0 "Q3" H 5050 2200 50  0000 L CNN
+F 1 "BC858CLT1G" H 4300 2100 50  0000 L CNN
+F 2 "Package_TO_SOT_SMD:SOT-23" H 5050 2300 50  0001 C CNN
+F 3 "~" H 4850 2200 50  0001 C CNN
+	1    4850 2200
+	1    0    0    1
+$EndComp
+Connection ~ 4950 2000
+Wire Wire Line
+	4950 2000 5250 2000
 $EndSCHEMATC
